File: Water_Valve_Sensor/Water_Valve_Sensor.sch (KiCad schematic (older format))
At the start: 30 parts, among them J1 Barrel_Jack, J2 WATER_PROBE, J3 SENSITIVITY_SELECTOR, J5 VALVE, Q1 Q_PMOS_DGS, U1 NE555D, U2 LM2904, U3 47U

Commit message: Fixed Wiring Issue
Added support for 2x6 header for Custom Setting Attachment
Parts:
- removed J3: SENSITIVITY_SELECTOR, Connector_PinHeader_2.54mm:PinHeader_2x05_P2.54mm_Vertical, symbol wickerlib:HEADER-MALE-10POS-TH-2x5-P0.1IN
- added J3: SENSITIVITY_SELECTOR, Connector_PinHeader_2.54mm:PinHeader_2x06_P2.54mm_Vertical, symbol Connector_Generic:Conn_02x06_Odd_Even
Connections:
- net +12V: now also J3.1 (Pin_1), J3.2 (Pin_2)
- net GND: now also J3.10 (Pin_10), J3.12 (Pin_12), J3.4 (Pin_4), J3.6 (Pin_6), J3.8 (Pin_8)
- net at R7.1: now also J3.3 (Pin_3)
- net at R3.1: now also J3.11 (Pin_11)
- net at R4.1: now also J3.9 (Pin_9)
- net at R5.1: now also J3.7 (Pin_7)
- net at R6.1: now also J3.5 (Pin_5)
Changed lines of the file:
@@
 	4300 2725 4300 2450
-$Comp
-L wickerlib:HEADER-MALE-10POS-TH-2x5-P0.1IN J3
-U 1 1 61470126
-P 3450 6550
-F 0 "J3" H 3450 6375 50  0000 C CNN
-F 1 "SENSITIVITY_SELECTOR" H 3450 6466 50  0000 C CNN
-F 2 "Connector_PinHeader_2.54mm:PinHeader_2x05_P2.54mm_Vertical" H 3450 6500 50  0001 C CIN
-F 3 "https://cdn.amphenol-icc.com/media/wysiwyg/files/drawing/67996.pdf" H 3400 6550 5   0001 C CNN
-F 4 "HEADER MALE 10POS TH 2x5 0.1IN" H 3450 6500 50  0001 C CIN "Description"
-F 5 "Amphenol" H 3450 6500 50  0001 C CIN "MF_Name"
-F 6 "67997-410HLF" H 3450 6500 50  0001 C CIN "MF_PN"
-F 7 "Digikey" H 3450 6500 50  0001 C CIN "S1_Name"
-F 8 "609-3243-ND" H 3450 6500 50  0001 C CIN "S1_PN"
-F 9 "500" H 3450 6500 50  0001 C CIN "XSize_mils"
-F 10 "200" H 3450 6500 50  0001 C CIN "YSize_mils"
-F 11 "th" H 3450 6500 50  0001 C CIN "Type"
-	1    3450 6550
-	-1   0    0    1
-$EndComp
 $Comp
 L Device:R R7
@@
 Wire Wire Line
 	6025 4150 5900 4150
+$Comp
+L Connector_Generic:Conn_02x06_Odd_Even J3
+U 1 1 612D4D1E
+P 3400 6700
+F 0 "J3" H 3450 7225 50  0000 C CNN
+F 1 "SENSITIVITY_SELECTOR" H 3450 7150 50  0000 C CNN
+F 2 "Connector_PinHeader_2.54mm:PinHeader_2x06_P2.54mm_Vertical" H 3400 6700 50  0001 C CNN
+F 3 "~" H 3400 6700 50  0001 C CNN
+	1    3400 6700
+	1    0    0    -1
+$EndComp
+$Comp
+L power:+12V #PWR0101
+U 1 1 612D79F2
+P 4050 6275
+F 0 "#PWR0101" H 4050 6125 50  0001 C CNN
+F 1 "+12V" H 4065 6448 50  0000 C CNN
+F 2 "" H 4050 6275 50  0001 C CNN
+F 3 "" H 4050 6275 50  0001 C CNN
+	1    4050 6275
+	1    0    0    -1
+$EndComp
+Wire Wire Line
+	4050 6275 4050 6375
+Wire Wire Line
+	4050 6375 3800 6375
+Wire Wire Line
+	3125 6500 3200 6500
+Wire Wire Line
+	3125 6375 3800 6375
+Wire Wire Line
+	3800 6375 3800 6500
+Wire Wire Line
+	3125 6375 3125 6500
+Wire Wire Line
+	3800 6500 3700 6500
+Connection ~ 3800 6375
 $EndSCHEMATC

Commit message: Changes to resistor selections
Updated sensitivty resistors.
Parts:
- J1: symbol Connector:Barrel_Jack -> Connector:Barrel_Jack_Switch
- R3: value 9K -> 383K
- R4: value 1K8 -> 255K
- R5: value 900R -> 127K
- R6: value 180R -> 63K4
- R7: value 91R -> 31K6
Connections:
- net +12V: no longer J3.1 (Pin_1)
- net GND: now also J1.3
- net R_SENSITIVITY: now also J3.1 (Pin_1)
Changed lines of the file:
@@
 $EndDescr
 $Comp
-L Connector:Barrel_Jack J1
+L Connector:Barrel_Jack_Switch J1
 U 1 1 61451CAE
 P 1825 2050
@@
 	2750 2875 2750 2825
 Wire Wire Line
-	2475 2150 2125 2150
+	2475 2150 2225 2150
 $Comp
 L Device:C C1
@@
 P 2975 6600
 F 0 "R7" V 2768 6600 50  0000 C CNN
-F 1 "91R" H 2859 6600 50  0000 C CNN
+F 1 "31K6" H 2859 6600 50  0000 C CNN
 F 2 "Resistor_THT:R_Axial_DIN0207_L6.3mm_D2.5mm_P7.62mm_Horizontal" V 2905 6600 50  0001 C CNN
 F 3 "~" H 2975 6600 50  0001 C CNN
@@
 P 2750 6700
 F 0 "R6" V 2543 6700 50  0000 C CNN
-F 1 "180R" H 2634 6700 50  0000 C CNN
+F 1 "63K4" H 2634 6700 50  0000 C CNN
 F 2 "Resistor_THT:R_Axial_DIN0207_L6.3mm_D2.5mm_P7.62mm_Horizontal" V 2680 6700 50  0001 C CNN
 F 3 "~" H 2750 6700 50  0001 C CNN
@@
 P 2525 6800
 F 0 "R5" V 2318 6800 50  0000 C CNN
-F 1 "900R" H 2409 6800 50  0000 C CNN
+F 1 "127K" H 2409 6800 50  0000 C CNN
 F 2 "Resistor_THT:R_Axial_DIN0207_L6.3mm_D2.5mm_P7.62mm_Horizontal" V 2455 6800 50  0001 C CNN
 F 3 "~" H 2525 6800 50  0001 C CNN
@@
 P 2300 6900
 F 0 "R4" V 2093 6900 50  0000 C CNN
-F 1 "1K8" H 2184 6900 50  0000 C CNN
+F 1 "255K" H 2184 6900 50  0000 C CNN
 F 2 "Resistor_THT:R_Axial_DIN0207_L6.3mm_D2.5mm_P7.62mm_Horizontal" V 2230 6900 50  0001 C CNN
 F 3 "~" H 2300 6900 50  0001 C CNN
@@
 P 2075 7000
 F 0 "R3" V 1868 7000 50  0000 C CNN
-F 1 "9K" H 1959 7000 50  0000 C CNN
+F 1 "383K" H 1959 7000 50  0000 C CNN
 F 2 "Resistor_THT:R_Axial_DIN0207_L6.3mm_D2.5mm_P7.62mm_Horizontal" V 2005 7000 50  0001 C CNN
 F 3 "~" H 2075 7000 50  0001 C CNN
@@
 L power:+12V #PWR0101
 U 1 1 612D79F2
-P 4050 6275
-F 0 "#PWR0101" H 4050 6125 50  0001 C CNN
-F 1 "+12V" H 4065 6448 50  0000 C CNN
-F 2 "" H 4050 6275 50  0001 C CNN
-F 3 "" H 4050 6275 50  0001 C CNN
-	1    4050 6275
-	1    0    0    -1
-$EndComp
-Wire Wire Line
-	4050 6275 4050 6375
-Wire Wire Line
-	4050 6375 3800 6375
-Wire Wire Line
-	3125 6500 3200 6500
-Wire Wire Line
-	3125 6375 3800 6375
-Wire Wire Line
-	3800 6375 3800 6500
-Wire Wire Line
-	3125 6375 3125 6500
-Wire Wire Line
-	3800 6500 3700 6500
-Connection ~ 3800 6375
+P 4050 6325
+F 0 "#PWR0101" H 4050 6175 50  0001 C CNN
+F 1 "+12V" H 4065 6498 50  0000 C CNN
+F 2 "" H 4050 6325 50  0001 C CNN
+F 3 "" H 4050 6325 50  0001 C CNN
+	1    4050 6325
+	1    0    0    -1
+$EndComp
+Wire Wire Line
+	4050 6325 4050 6500
+Wire Wire Line
+	2125 2050 2225 2050
+Wire Wire Line
+	2225 2050 2225 2150
+Connection ~ 2225 2150
+Wire Wire Line
+	2225 2150 2125 2150
+Wire Wire Line
+	3700 6500 4050 6500
+Wire Wire Line
+	1775 6500 3200 6500
+Wire Wire Line
+	1775 6500 1775 6600
+Connection ~ 1775 6600
 $EndSCHEMATC
